File: Individual motor driver/Individual motor driver.sch (KiCad schematic (older format))
At the start: 7 parts

Commit message: New PCB project
Parts:
- removed P? (x3): CONN_01X02, symbol CONN_01X02
- added C1, C2, C3, C4: 0.01uF, Capacitor_THT:C_Axial_L3.8mm_D2.6mm_P7.50mm_Horizontal, symbol C
- added D1, D2, D3: Led_Small, LED_THT:LED_D3.0mm, symbol Led_Small
- added P2, P3, P4, P5, P6, P8: CONN_01X02, Connector_PinHeader_2.54mm:PinHeader_1x02_P2.54mm_Vertical, symbol CONN_01X02
- added P7: CONN_01X04, Connector_PinHeader_2.54mm:PinHeader_1x04_P2.54mm_Vertical, symbol CONN_01X04
- added Q1, Q2, Q3, Q4: PN2222A, Package_TO_SOT_THT:TO-92_Inline, symbol PN2222A
- added R1: 100, Resistor_THT:R_Axial_Power_L20.0mm_W6.4mm_P5.08mm_Vertical, symbol R
- added R10, R2, R3, R4, R5, R7, R8, R9: 10k, Resistor_THT:R_Axial_Power_L20.0mm_W6.4mm_P5.08mm_Vertical, symbol R
- added R11, R6: 50, Resistor_THT:R_Axial_Power_L20.0mm_W6.4mm_P5.08mm_Vertical, symbol R
- added U3, U4: ACS711xLCTR-12AB, Package_SO:SOIC-8_3.9x4.9mm_P1.27mm, symbol ACS711xLCTR-12AB
- Motor1: renamed from Motor; footprint DIL16 -> Package_DIP:DIP-16_W7.62mm
- P1: renamed from P?; footprint (none) -> Connector_PinHeader_2.54mm:PinHeader_1x02_P2.54mm_Vertical
- gave numbers to parts that had none: 2
Connections:
- net 5V: now also P6.1 (P1), Q1.3 (C), Q2.3 (C), Q3.3 (C), Q4.3 (C), R2.2, R3.2, R7.2, R8.2
- net GND: now also U1.39 (GND), U2.39 (GND), C1.1, C2.1, C3.1, C4.1, D1.1 (K), P2.2 (P2), P5.2 (P2), P6.2 (P2), P8.2 (P2), R11.1, R6.1, U3.5 (GND), U4.5 (GND)
- net Rotary_Encoder_1A: now also U2.23 (PB14_MISO2), R10.2; no longer P1.1 (P1)
- net Rotary_Encoder_1B: now also U2.24 (PB15_MOSI2), R9.1; no longer P1.2 (P2)
- net Rotary_Encoder_2A: now also U1.23 (PB14_MISO2), R5.2
- net Rotary_Encoder_2B: now also U1.24 (PB15_MOSI2), R4.1
- net at U1.13 (PB0): now also Q2.2 (B)
- net at U1.14 (PB1): now also Q1.2 (B)
- net SCL: now reaches U1.34 (PB6_SCL1)
- net SCL: now also U2.34 (PB6_SCL1), P3.2 (P2)
- net SDA: now reaches U1.35 (PB7_SDA1)
- net SDA: now also U2.35 (PB7_SDA1), P3.1 (P1)
- net Stall_2: now reaches U1.4 (PC15)
- net Stall_2: now also D2.2 (A)
- net 3.3v: now reaches U1.40 (VCC3V3)
- net 3.3v: now also U2.40 (VCC3V3), U3.8 (VCC), U4.8 (VCC)
- net Limit2: now reaches U1.5 (PA0)
- net Limit2: now also P2.1 (P1)
- net M2:Current: now reaches U1.6 (PA1)
- net M2:Current: now also U4.7 (VIOUT)
- net M2:C2: now reaches Motor1.10 (3A)
- net M2:C2: now also Q1.1 (E)
- net M2:O2: now reaches Motor1.11 (3Y)
- net M2:O2: now also U4.3 (IP-), U4.4 (IP-)
- net M2:O1: now reaches Motor1.14 (4Y)
- net M2:O1: now also P7.3 (P3)
- net M2:C1: now reaches Motor1.15 (4A)
- net M2:C1: now also Q2.1 (E)
- net M1:C1: now reaches Motor1.2 (1A)
- net M1:C1: now also Q4.1 (E)
- net M1:O1: now reaches Motor1.3 (1Y)
- net M1:O1: now also U3.1 (IP+), U3.2 (IP+)
- net M1:O2: now reaches Motor1.6 (2Y)
- net M1:O2: now also P7.2 (P2)
- net M1:C2: now reaches Motor1.7 (2A)
- net M1:C2: now also Q3.1 (E)
- net VCC: now reaches Motor1.8 (VCC2)
- net VCC: now also P5.1 (P1), R1.2
- net at U2.13 (PB0): now also Q4.2 (B)
- net at U2.14 (PB1): now also Q3.2 (B)
- net Stall_1: now reaches U2.4 (PC15)
- net Stall_1: now also D3.2 (A)
- net Limit1: now reaches U2.5 (PA0)
- net Limit1: now also P8.1 (P1)
- net M1:Current: now reaches U2.6 (PA1)
- net M1:Current: now also U3.7 (VIOUT)
- new net: C1.2, P1.1 (P1), R2.1, R4.2
- new net: C2.2, P1.2 (P2), R3.1, R5.1
- new net: P7.1 (P1), U3.3 (IP-), U3.4 (IP-)
- new net: P7.4 (P4), U4.1 (IP+), U4.2 (IP+)
- new net: D1.2 (A), R1.1
- new net: D3.1 (K), R11.2
- new net: D2.1 (K), R6.2
- new net: C3.2, P4.1 (P1), R7.1, R9.2
- new net: C4.2, P4.2 (P2), R10.1, R8.1
Other:
- moved on the sheet: Motor1, P1, U1, U2

Commit message: PCB updates
Parts:
- added P9: CONN_01X02, Connector_PinHeader_2.54mm:PinHeader_1x02_P2.54mm_Vertical, symbol CONN_01X02
Connections:
- net SCL: now also P9.2 (P2)
- net SDA: now also P9.1 (P1)
Changed lines of the file:
@@
 Wire Wire Line
 	1450 3650 1450 3350
+$Comp
+L CONN_01X02 P9
+U 1 1 5BED8ED6
+P 6000 7000
+F 0 "P9" H 6000 7150 50  0000 C CNN
+F 1 "CONN_01X02" V 6100 7000 50  0000 C CNN
+F 2 "Connector_PinHeader_2.54mm:PinHeader_1x02_P2.54mm_Vertical" H 6000 7000 50  0001 C CNN
+F 3 "" H 6000 7000 50  0000 C CNN
+	1    6000 7000
+	0    -1   -1   0
+$EndComp
+Wire Wire Line
+	5950 7200 5950 7300
+Connection ~ 5950 7300
+Wire Wire Line
+	6050 7200 6050 7350
+Wire Wire Line
+	6050 7350 5950 7350
+Wire Wire Line
+	5950 7350 5950 7400
+Connection ~ 5950 7400
 $EndSCHEMATC

Commit message: Fixed rotary encoder filter
Connections:
- net 3.3v: now also R2.2, R3.2, R7.2, R8.2
- net 5V: no longer R2.2, R3.2, R7.2, R8.2
- net Rotary_Encoder_1A: now also C4.2
- net Rotary_Encoder_1B: now also C3.2
- net Rotary_Encoder_2A: now also C2.2
- net Rotary_Encoder_2B: now also C1.2
- net at P1.1 (P1), R2.1, R4.2: no longer C1.2
- net at P1.2 (P2), R3.1, R5.1: no longer C2.2
- net at P4.1 (P1), R7.1, R9.2: no longer C3.2
- net at P4.2 (P2), R10.1, R8.1: no longer C4.2
Changed lines of the file:
@@
 Text GLabel 1250 3650 2    60   Input ~ 0
-5V
-Text GLabel 2100 5550 0    60   Input ~ 0
 5V
 $Comp
@@
 Text GLabel 5850 4850 0    60   Input ~ 0
 Rotary_Encoder_1B
-Text GLabel 5450 5550 0    60   Input ~ 0
-5V
 $Comp
 L R R7
@@
 	2800 5100 2750 5100
 Wire Wire Line
-	2750 5100 2750 5250
-Wire Wire Line
-	2750 5250 2600 5250
-Wire Wire Line
-	2800 5950 2800 5850
-Wire Wire Line
-	2800 5850 2600 5850
-Wire Wire Line
 	3100 5100 3250 5100
 Wire Wire Line
@@
 Wire Wire Line
 	6150 5100 6100 5100
-Wire Wire Line
-	6100 5100 6100 5250
-Wire Wire Line
-	6100 5250 5950 5250
-Wire Wire Line
-	6150 5950 6150 5850
-Wire Wire Line
-	6150 5850 5950 5850
 Wire Wire Line
 	6450 5100 6600 5100
@@
 	5950 7350 5950 7400
 Connection ~ 5950 7400
+Text GLabel 5450 5550 0    60   Input ~ 0
+3.3v
+Text GLabel 2100 5550 0    60   Input ~ 0
+3.3v
+Wire Wire Line
+	6100 5100 6100 4900
+Wire Wire Line
+	6100 4900 5950 4900
+Connection ~ 5950 4900
+Wire Wire Line
+	6150 5950 6150 6200
+Wire Wire Line
+	6150 6200 5950 6200
+Connection ~ 5950 6200
+Wire Wire Line
+	2750 5100 2750 4900
+Wire Wire Line
+	2750 4900 2600 4900
+Connection ~ 2600 4900
+Wire Wire Line
+	2800 5950 2750 5950
+Wire Wire Line
+	2750 5950 2750 6200
+Wire Wire Line
+	2750 6200 2600 6200
+Connection ~ 2600 6200
 $EndSCHEMATC
